Commit message: add controller mesh, fix infinite loop in IK

File: urdf/02-oculus.urdf (robot description, URDF)
Before this commit: robot oculus, 3 links, 2 joints
Links:
- link oculus_right_controller: geometry visual mesh filename=package://pepper_surrogate/meshes/right_touch_controller.dae scale=0.012 0.012 0.012
