Commit message: both arms working

File: urdf/01-virtualarm.urdf (robot description, URDF)
Before this commit: robot virtualarm, 6 links, 5 joints
Links:
- added link l_gripper, mass 2e-06
- added link virtualarm_LBicep, mass 0.50527; collision mesh filename=package://pepper_meshes/meshes/1.0/LShoulderRoll_0.10.stl scale=0.1 0.1 0.1; visual mesh filename=package://pepper_meshes/meshes/1.0/LShoulderRoll.dae scale=0.1 0.1 0.1
- added link virtualarm_LElbow, mass 0.27495; collision mesh filename=package://pepper_meshes/meshes/1.0/LElbowYaw_0.10.stl scale=0.1 0.1 0.1; visual mesh filename=package://pepper_meshes/meshes/1.0/LElbowYaw.dae scale=0.1 0.1 0.1
- added link virtualarm_LForeArm, mass 0.16579; collision mesh filename=package://pepper_meshes/meshes/1.0/LElbowRoll_0.10.stl scale=0.1 0.1 0.1; visual mesh filename=package://pepper_meshes/meshes/1.0/LElbowRoll.dae scale=0.1 0.1 0.1
- added link virtualarm_LShoulder, mass 0.3125; collision mesh filename=package://pepper_meshes/meshes/1.0/LShoulderPitch_0.10.stl scale=0.1 0.1 0.1; visual mesh filename=package://pepper_meshes/meshes/1.0/LShoulderPitch.dae scale=0.1 0.1 0.1
- added link virtualarm_LTorso; visual sphere radius=0.05
- added link virtualarm_RTorso; visual sphere radius=0.05
- added link virtualarm_TorsoCenter; visual sphere radius=0.05
- added link virtualarm_l_wrist, mass 0.27555; collision mesh filename=package://pepper_meshes/meshes/1.0/LWristYaw_0.10.stl scale=0.1 0.1 0.1; visual mesh filename=package://pepper_meshes/meshes/1.0/LWristYaw.dae scale=0.1 0.1 0.1
Joints:
- added joint virtualarm_LElbowRoll: type revolute, parent virtualarm_LElbow, child virtualarm_LForeArm, origin xyz=0 0 0 rpy=0 0 0, axis 0 0 1.0, limit lower=0.00872665 upper=1.56207 effort=2.666 velocity=9.22756
- added joint virtualarm_LElbowYaw: type revolute, parent virtualarm_LBicep, child virtualarm_LElbow, origin xyz=0.1812 -0.015 0.00013 rpy=0 -0.157079 0, axis 1.0 0 0, limit lower=-2.08567 upper=2.08567 effort=5.428 velocity=7.33998
- added joint virtualarm_LHand: type revolute, parent virtualarm_l_wrist, child l_gripper, origin xyz=0.025 0 0 rpy=0 0 0, axis 1.0 0 0, limit lower=0.02 upper=0.98 effort=0.144 velocity=12.56
- added joint virtualarm_LOmoplata: type revolute, parent virtualarm_LTorso, child virtualarm_LShoulder, origin xyz=0 0 0 rpy=0 0 0, axis 0 0 1.0, limit lower=-1.56207 upper=-0.00872665 effort=2.666 velocity=9.22756
- added joint virtualarm_LShoulderRoll: type revolute, parent virtualarm_LShoulder, child virtualarm_LBicep, origin xyz=0 0 0 rpy=0 0 0, axis 0 0 1.0, limit lower=-1.56207 upper=-0.00872665 effort=2.666 velocity=9.22756
- added joint virtualarm_LTorsoError: type revolute, parent virtualarm_TorsoCenter, child virtualarm_LTorso, origin xyz=0 0 0 rpy=0 0 0, axis 0 0 1.0, limit lower=-1.56207 upper=-0.00872665 effort=2.666 velocity=9.22756
- added joint virtualarm_LWristYaw: type revolute, parent virtualarm_LForeArm, child virtualarm_l_wrist, origin xyz=0.15 0 0 rpy=0 0 0, axis 1.0 0 0, limit lower=-1.82387 upper=1.82387 effort=0.2014 velocity=17.3835
- added joint virtualarm_ROmoplata: type revolute, parent virtualarm_RTorso, child virtualarm_RShoulder, origin xyz=0 0 0 rpy=0 0 0, axis 0 0 1.0, limit lower=-1.56207 upper=-0.00872665 effort=2.666 velocity=9.22756
- added joint virtualarm_RTorsoError: type revolute, parent virtualarm_TorsoCenter, child virtualarm_RTorso, origin xyz=0 0 0 rpy=0 0 0, axis 0 0 1.0, limit lower=-1.56207 upper=-0.00872665 effort=2.666 velocity=9.22756

File: urdf/02-oculus.urdf (robot description, URDF)
Before this commit: robot oculus, 3 links, 2 joints
Links:
- added link oculus_left_controller; visual mesh filename=package://pepper_surrogate/meshes/left_touch_controller.dae scale=0.012 0.012 0.012
- added link oculus_left_vrhand; visual mesh filename=package://pepper_surrogate/meshes/Hand.dae scale=0.05 -0.05 0.05
- link oculus: geometry visual mesh filename=package://pepper_surrogate/meshes/oculus_rift.dae scale=0.0002 0.0002 0.0002
Joints:
- removed joint oculus_to_rcontroller
- added joint left_controller_to_left_vrhand: type revolute, parent oculus_left_controller, child oculus_left_vrhand, origin xyz=0 0 0 rpy=0 0 0, axis 0 0 1.0, limit lower=-1.56207 upper=-0.00872665 effort=2.666 velocity=9.22756
- added joint oculus_to_left_controller: type revolute, parent oculus, child oculus_left_controller, origin xyz=0 0 0 rpy=0 0 0, axis 0 0 1.0, limit lower=-1.56207 upper=-0.00872665 effort=2.666 velocity=9.22756
- added joint oculus_to_right_controller: type revolute, parent oculus, child oculus_right_controller, origin xyz=0 0 0 rpy=0 0 0, axis 0 0 1.0, limit lower=-1.56207 upper=-0.00872665 effort=2.666 velocity=9.22756
