Commit message: arm scale

File: urdf/01-virtualarm.xacro (robot description, xacro)
@@ -1,4 +1,5 @@
 <?xml version="1.0"?>
-<robot name="virtualarm">
+<robot name="virtualarm" xmlns:xacro="http://ros.org/wiki/xacro">
+  <xacro:property name="scale" value="1.8" />
   <link name="virtualarm_TorsoCenter">
     <visual>
@@ -39,11 +40,11 @@
     <visual>
       <geometry>
-        <mesh filename="package://pepper_meshes/meshes/1.0/RShoulderPitch.dae" scale="0.1 0.1 0.1"/>
-      </geometry>
-      <origin rpy="0 0 0" xyz="0 0 0"/>
-    </visual>
-    <collision>
-      <geometry>
-        <mesh filename="package://pepper_meshes/meshes/1.0/RShoulderPitch_0.10.stl" scale="0.1 0.1 0.1"/>
+        <mesh filename="package://pepper_meshes/meshes/1.0/RShoulderPitch.dae" scale="${0.1*scale} ${0.1*scale} ${0.1*scale}"/>
+      </geometry>
+      <origin rpy="0 0 0" xyz="0 0 0"/>
+    </visual>
+    <collision>
+      <geometry>
+        <mesh filename="package://pepper_meshes/meshes/1.0/RShoulderPitch_0.10.stl" scale="${0.1*scale} ${0.1*scale} ${0.1*scale}"/>
       </geometry>
       <origin rpy="0 0 0" xyz="0 0 0"/>
@@ -65,11 +66,11 @@
     <visual>
       <geometry>
-        <mesh filename="package://pepper_meshes/meshes/1.0/RShoulderRoll.dae" scale="0.1 0.1 0.1"/>
-      </geometry>
-      <origin rpy="0 0 0" xyz="0 0 0"/>
-    </visual>
-    <collision>
-      <geometry>
-        <mesh filename="package://pepper_meshes/meshes/1.0/RShoulderRoll_0.10.stl" scale="0.1 0.1 0.1"/>
+        <mesh filename="package://pepper_meshes/meshes/1.0/RShoulderRoll.dae" scale="${0.1*scale} ${0.1*scale} ${0.1*scale}"/>
+      </geometry>
+      <origin rpy="0 0 0" xyz="0 0 0"/>
+    </visual>
+    <collision>
+      <geometry>
+        <mesh filename="package://pepper_meshes/meshes/1.0/RShoulderRoll_0.10.stl" scale="${0.1*scale} ${0.1*scale} ${0.1*scale}"/>
       </geometry>
       <origin rpy="0 0 0" xyz="0 0 0"/>
@@ -91,11 +92,11 @@
     <visual>
       <geometry>
-        <mesh filename="package://pepper_meshes/meshes/1.0/RElbowYaw.dae" scale="0.1 0.1 0.1"/>
-      </geometry>
-      <origin rpy="0 0 0" xyz="0 0 0"/>
-    </visual>
-    <collision>
-      <geometry>
-        <mesh filename="package://pepper_meshes/meshes/1.0/RElbowYaw_0.10.stl" scale="0.1 0.1 0.1"/>
+        <mesh filename="package://pepper_meshes/meshes/1.0/RElbowYaw.dae" scale="${0.1*scale} ${0.1*scale} ${0.1*scale}"/>
+      </geometry>
+      <origin rpy="0 0 0" xyz="0 0 0"/>
+    </visual>
+    <collision>
+      <geometry>
+        <mesh filename="package://pepper_meshes/meshes/1.0/RElbowYaw_0.10.stl" scale="${0.1*scale} ${0.1*scale} ${0.1*scale}"/>
       </geometry>
       <origin rpy="0 0 0" xyz="0 0 0"/>
@@ -117,11 +118,11 @@
     <visual>
       <geometry>
-        <mesh filename="package://pepper_meshes/meshes/1.0/RElbowRoll.dae" scale="0.1 0.1 0.1"/>
-      </geometry>
-      <origin rpy="0 0 0" xyz="0 0 0"/>
-    </visual>
-    <collision>
-      <geometry>
-        <mesh filename="package://pepper_meshes/meshes/1.0/RElbowRoll_0.10.stl" scale="0.1 0.1 0.1"/>
+        <mesh filename="package://pepper_meshes/meshes/1.0/RElbowRoll.dae" scale="${0.1*scale} ${0.1*scale} ${0.1*scale}"/>
+      </geometry>
+      <origin rpy="0 0 0" xyz="0 0 0"/>
+    </visual>
+    <collision>
+      <geometry>
+        <mesh filename="package://pepper_meshes/meshes/1.0/RElbowRoll_0.10.stl" scale="${0.1*scale} ${0.1*scale} ${0.1*scale}"/>
       </geometry>
       <origin rpy="0 0 0" xyz="0 0 0"/>
@@ -143,11 +144,11 @@
     <visual>
       <geometry>
-        <mesh filename="package://pepper_meshes/meshes/1.0/RWristYaw.dae" scale="0.1 0.1 0.1"/>
-      </geometry>
-      <origin rpy="0 0 0" xyz="0 0 0"/>
-    </visual>
-    <collision>
-      <geometry>
-        <mesh filename="package://pepper_meshes/meshes/1.0/RWristYaw_0.10.stl" scale="0.1 0.1 0.1"/>
+        <mesh filename="package://pepper_meshes/meshes/1.0/RWristYaw.dae" scale="${0.1*scale} ${0.1*scale} ${0.1*scale}"/>
+      </geometry>
+      <origin rpy="0 0 0" xyz="0 0 0"/>
+    </visual>
+    <collision>
+      <geometry>
+        <mesh filename="package://pepper_meshes/meshes/1.0/RWristYaw_0.10.stl" scale="${0.1*scale} ${0.1*scale} ${0.1*scale}"/>
       </geometry>
       <origin rpy="0 0 0" xyz="0 0 0"/>
@@ -197,11 +198,11 @@
     <visual>
       <geometry>
-        <mesh filename="package://pepper_meshes/meshes/1.0/LShoulderPitch.dae" scale="0.1 0.1 0.1"/>
-      </geometry>
-      <origin rpy="0 0 0" xyz="0 0 0"/>
-    </visual>
-    <collision>
-      <geometry>
-        <mesh filename="package://pepper_meshes/meshes/1.0/LShoulderPitch_0.10.stl" scale="0.1 0.1 0.1"/>
+        <mesh filename="package://pepper_meshes/meshes/1.0/LShoulderPitch.dae" scale="${0.1*scale} ${0.1*scale} ${0.1*scale}"/>
+      </geometry>
+      <origin rpy="0 0 0" xyz="0 0 0"/>
+    </visual>
+    <collision>
+      <geometry>
+        <mesh filename="package://pepper_meshes/meshes/1.0/LShoulderPitch_0.10.stl" scale="${0.1*scale} ${0.1*scale} ${0.1*scale}"/>
       </geometry>
       <origin rpy="0 0 0" xyz="0 0 0"/>
@@ -223,11 +224,11 @@
     <visual>
       <geometry>
-        <mesh filename="package://pepper_meshes/meshes/1.0/LShoulderRoll.dae" scale="0.1 0.1 0.1"/>
-      </geometry>
-      <origin rpy="0 0 0" xyz="0 0 0"/>
-    </visual>
-    <collision>
-      <geometry>
-        <mesh filename="package://pepper_meshes/meshes/1.0/LShoulderRoll_0.10.stl" scale="0.1 0.1 0.1"/>
+        <mesh filename="package://pepper_meshes/meshes/1.0/LShoulderRoll.dae" scale="${0.1*scale} ${0.1*scale} ${0.1*scale}"/>
+      </geometry>
+      <origin rpy="0 0 0" xyz="0 0 0"/>
+    </visual>
+    <collision>
+      <geometry>
+        <mesh filename="package://pepper_meshes/meshes/1.0/LShoulderRoll_0.10.stl" scale="${0.1*scale} ${0.1*scale} ${0.1*scale}"/>
       </geometry>
       <origin rpy="0 0 0" xyz="0 0 0"/>
@@ -249,11 +250,11 @@
     <visual>
       <geometry>
-        <mesh filename="package://pepper_meshes/meshes/1.0/LElbowYaw.dae" scale="0.1 0.1 0.1"/>
-      </geometry>
-      <origin rpy="0 0 0" xyz="0 0 0"/>
-    </visual>
-    <collision>
-      <geometry>
-        <mesh filename="package://pepper_meshes/meshes/1.0/LElbowYaw_0.10.stl" scale="0.1 0.1 0.1"/>
+        <mesh filename="package://pepper_meshes/meshes/1.0/LElbowYaw.dae" scale="${0.1*scale} ${0.1*scale} ${0.1*scale}"/>
+      </geometry>
+      <origin rpy="0 0 0" xyz="0 0 0"/>
+    </visual>
+    <collision>
+      <geometry>
+        <mesh filename="package://pepper_meshes/meshes/1.0/LElbowYaw_0.10.stl" scale="${0.1*scale} ${0.1*scale} ${0.1*scale}"/>
       </geometry>
       <origin rpy="0 0 0" xyz="0 0 0"/>
@@ -275,11 +276,11 @@
     <visual>
       <geometry>
-        <mesh filename="package://pepper_meshes/meshes/1.0/LElbowRoll.dae" scale="0.1 0.1 0.1"/>
-      </geometry>
-      <origin rpy="0 0 0" xyz="0 0 0"/>
-    </visual>
-    <collision>
-      <geometry>
-        <mesh filename="package://pepper_meshes/meshes/1.0/LElbowRoll_0.10.stl" scale="0.1 0.1 0.1"/>
+        <mesh filename="package://pepper_meshes/meshes/1.0/LElbowRoll.dae" scale="${0.1*scale} ${0.1*scale} ${0.1*scale}"/>
+      </geometry>
+      <origin rpy="0 0 0" xyz="0 0 0"/>
+    </visual>
+    <collision>
+      <geometry>
+        <mesh filename="package://pepper_meshes/meshes/1.0/LElbowRoll_0.10.stl" scale="${0.1*scale} ${0.1*scale} ${0.1*scale}"/>
       </geometry>
       <origin rpy="0 0 0" xyz="0 0 0"/>
@@ -301,11 +302,11 @@
     <visual>
       <geometry>
-        <mesh filename="package://pepper_meshes/meshes/1.0/LWristYaw.dae" scale="0.1 0.1 0.1"/>
-      </geometry>
-      <origin rpy="0 0 0" xyz="0 0 0"/>
-    </visual>
-    <collision>
-      <geometry>
-        <mesh filename="package://pepper_meshes/meshes/1.0/LWristYaw_0.10.stl" scale="0.1 0.1 0.1"/>
+        <mesh filename="package://pepper_meshes/meshes/1.0/LWristYaw.dae" scale="${0.1*scale} ${0.1*scale} ${0.1*scale}"/>
+      </geometry>
+      <origin rpy="0 0 0" xyz="0 0 0"/>
+    </visual>
+    <collision>
+      <geometry>
+        <mesh filename="package://pepper_meshes/meshes/1.0/LWristYaw_0.10.stl" scale="${0.1*scale} ${0.1*scale} ${0.1*scale}"/>
       </geometry>
       <origin rpy="0 0 0" xyz="0 0 0"/>

Commit message: adds grippers

File: urdf/01-virtualarm.xacro (robot description, xacro)
@@ -157,14 +157,20 @@
   <joint name="virtualarm_RHand" type="revolute">
     <parent link="virtualarm_r_wrist"/>
-    <child link="r_gripper"/>
+    <child link="virtualarm_r_gripper"/>
     <origin rpy="0 0 0" xyz="0.025 0 0"/>
     <axis xyz="1.0 0 0"/>
     <limit effort="0.144" lower="0.02" upper="0.98" velocity="12.56"/>
   </joint>
-  <link name="r_gripper">
+  <link name="virtualarm_r_gripper">
     <inertial>
       <mass value="2e-06"/>
       <inertia ixx="1.1e-09" ixy="0" ixz="0" iyy="1.1e-09" iyz="0" izz="1.1e-09"/>
     </inertial>
+    <visual>
+      <geometry>
+        <cylinder radius="0.01" length="0.06"/>
+      </geometry>
+      <origin rpy="0 0 0" xyz="0 0 0"/>
+    </visual>
   </link>
   <joint name="virtualarm_LTorsoError" type="revolute">
@@ -315,14 +321,20 @@
   <joint name="virtualarm_LHand" type="revolute">
     <parent link="virtualarm_l_wrist"/>
-    <child link="l_gripper"/>
+    <child link="virtualarm_l_gripper"/>
     <origin rpy="0 0 0" xyz="0.025 0 0"/>
     <axis xyz="1.0 0 0"/>
     <limit effort="0.144" lower="0.02" upper="0.98" velocity="12.56"/>
   </joint>
-  <link name="l_gripper">
+  <link name="virtualarm_l_gripper">
     <inertial>
       <mass value="2e-06"/>
       <inertia ixx="1.1e-09" ixy="0" ixz="0" iyy="1.1e-09" iyz="0" izz="1.1e-09"/>
     </inertial>
+    <visual>
+      <geometry>
+        <cylinder radius="0.01" length="0.06"/>
+      </geometry>
+      <origin rpy="0 0 0" xyz="0 0 0"/>
+    </visual>
   </link>
 </robot>

Commit message: gripper control

File: urdf/01-virtualarm.xacro (robot description, xacro)
@@ -171,5 +171,5 @@
         <cylinder radius="0.01" length="0.06"/>
       </geometry>
-      <origin rpy="0 0 0" xyz="0 0 0"/>
+      <origin rpy="0 0 0" xyz="0 0 -0.03"/>
     </visual>
   </link>
@@ -335,5 +335,5 @@
         <cylinder radius="0.01" length="0.06"/>
       </geometry>
-      <origin rpy="0 0 0" xyz="0 0 0"/>
+      <origin rpy="0 0 0" xyz="0 0 -0.03"/>
     </visual>
   </link>
